File: TRS80_Floppy_Adapter.kicad_sch (KiCad schematic)
At the start: 21 parts, among them J1 Conn_02x01, J2 Conn_01x03_Socket, J3 Conn_02x01, J4 Conn_01x03, J5 Conn_01x03, J6 Conn_01x03_Socket, U1 74LS32, U2 74LS32

Commit message: Add files via upload
Parts:
- removed U2: 74LS32, symbol 74xx:74LS32
- added unit 3 of U1
- added unit 1 of U1
- added unit 2 of U1
- added unit 4 of U1
- C1: footprint (none) -> GenericComponents:Capcitor Radial .200
- D1, D2, D3, D4, J1, J3: footprint (none) -> Connector_PinHeader_2.54mm:PinHeader_1x02_P2.54mm_Vertical
- J2, J6: footprint (none) -> Connector_PinSocket_2.54mm:PinSocket_1x03_P2.54mm_Vertical
- J4, J5: footprint (none) -> Connector_PinHeader_2.54mm:PinHeader_1x03_P2.54mm_Vertical
- R1, R2, R3, R4: footprint (none) -> GenericComponents:Resistor-.4in
- U1: footprint (none) -> GenericComponents:DIP-14pin
- renumbered PC_5inch to PC_5inch1, TRS80-5inch to TRS80-5inch1, TRS80_8inch to TRS80_8inch1
Connections:
- net at TRS80-5inch1.16 (Pin_16), TRS80_8inch1.18 (Pin_18): now also U1.1, U1.12, U1.4, U1.9
- net at PC_5inch2.14 (Pin_14), TRS80-5inch1.10 (Pin_10), TRS80_8inch1.26 (Pin_26): now also U1.2
- net at PC_5inch2.12 (Pin_12), TRS80-5inch1.12 (Pin_12), TRS80_8inch1.28 (Pin_28): now also U1.5
- net at PC_5inch1.14 (Pin_14), TRS80-5inch1.14 (Pin_14), TRS80_8inch1.30 (Pin_30): now also U1.10
- net at PC_5inch1.12 (Pin_12), TRS80-5inch1.32 (Pin_32), TRS80_8inch1.32 (Pin_32): now also U1.13
- net at PC_5inch1.10 (Pin_10): now also U1.8
- net at PC_5inch1.16 (Pin_16): now also U1.11
- net at PC_5inch2.10 (Pin_10): now also U1.3
- net at PC_5inch2.16 (Pin_16): now also U1.6

Commit message: Add files via upload
Parts:
- R1, R2, R3, R4: footprint GenericComponents:Resistor-.4in -> Resistor_THT:R_Axial_DIN0204_L3.6mm_D1.6mm_P7.62mm_Horizontal
- renumbered J3 to J2, J2 to J3, J6 to J4, J4 to J5, J5 to J6
Other:
- moved on the sheet: J2
Changed lines of the file:
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@@
 	(text "Power In"
 		(exclude_from_sim no)
-		(at 234.188 62.738 0)
+		(at 197.358 -21.082 0)
 		(effects
 			(font
@@
 		(on_board yes)
 		(dnp no)
-		(property "Reference" "J6"
+		(property "Reference" "J4"
 			(at 125.73 168.9099 0)
 			(effects
@@
 			(project "TRS80M2 50-34 Floppy Adapter"
 				(path "/f29434cd-fd41-45dc-9c32-41e112fe785e"
-					(reference "J6")
+					(reference "J4")
 					(unit 1)
 				)
@@
 	(symbol
 		(lib_id "power:+5V")
-		(at 226.06 68.58 0)
+		(at 189.23 -15.24 0)
 		(unit 1)
 		(exclude_from_sim no)
@@
 		(dnp no)
 		(property "Reference" "#PWR012"
-			(at 226.06 72.39 0)
+			(at 189.23 -11.43 0)
 			(effects
 				(font
@@
 		)
 		(property "Value" "+5V"
-			(at 226.06 63.5 0)
+			(at 189.23 -20.32 0)
 			(effects
 				(font
@@
 		)
 		(property "Footprint" ""
-			(at 226.06 68.58 0)
+			(at 189.23 -15.24 0)
 			(effects
 				(font
@@
 		)
 		(property "Datasheet" ""
-			(at 226.06 68.58 0)
+			(at 189.23 -15.24 0)
 			(effects
 				(font
@@
 		)
 		(property "Description" "Power symbol creates a global label with name \"+5V\""
-			(at 226.06 68.58 0)
+			(at 189.23 -15.24 0)
 			(effects
 				(font
@@
 	(symbol
 		(lib_id "Connector_Generic:Conn_02x01")
-		(at 231.14 68.58 0)
-		(unit 1)
-		(exclude_from_sim no)
-		(in_bom yes)
-		(on_board yes)
-		(dnp no)
-		(property "Reference" "J3"
-			(at 232.41 66.04 0)
+		(at 194.31 -15.24 0)
+		(unit 1)
+		(exclude_from_sim no)
+		(in_bom yes)
+		(on_board yes)
+		(dnp no)
+		(property "Reference" "J2"
+			(at 195.58 -15.24 0)
 			(effects
 				(font
@@
 		)
 		(property "Value" "Conn_02x01"
-			(at 232.41 64.77 0)
+			(at 195.58 -19.05 0)
 			(effects
 				(font
@@
 		)
 		(property "Footprint" "Connector_PinHeader_2.54mm:PinHeader_1x02_P2.54mm_Vertical"
-			(at 231.14 68.58 0)
+			(at 194.31 -15.24 0)
 			(effects
 				(font
@@
 		)
 		(property "Datasheet" "~"
-			(at 231.14 68.58 0)
+			(at 194.31 -15.24 0)
 			(effects
 				(font
@@
 		)
 		(property "Description" "Generic connector, double row, 02x01, this symbol is compatible with counter-clockwise, top-bottom and odd-even numbering schemes., script generated (kicad-library-utils/schlib/autogen/connector/)"
-			(at 231.14 68.58 0)
+			(at 194.31 -15.24 0)
 			(effects
 				(font
@@
 			(project "TRS80M2 50-34 Floppy Adapter"
 				(path "/f29434cd-fd41-45dc-9c32-41e112fe785e"
-					(reference "J3")
+					(reference "J2")
 					(unit 1)
 				)
@@
 			)
 		)
-		(property "Footprint" "GenericComponents:Resistor-.4in"
+		(property "Footprint" "Resistor_THT:R_Axial_DIN0204_L3.6mm_D1.6mm_P7.62mm_Horizontal"
 			(at 138.938 149.098 90)
 			(effects
@@
 		(on_board yes)
 		(dnp no)
-		(property "Reference" "J2"
+		(property "Reference" "J3"
 			(at 125.73 151.1299 0)
 			(effects
@@
 			(project "TRS80M2 50-34 Floppy Adapter"
 				(path "/f29434cd-fd41-45dc-9c32-41e112fe785e"
-					(reference "J2")
+					(reference "J3")
 					(unit 1)
 				)
@@
 			)
 		)
-		(property "Footprint" "GenericComponents:Resistor-.4in"
+		(property "Footprint" "Resistor_THT:R_Axial_DIN0204_L3.6mm_D1.6mm_P7.62mm_Horizontal"
 			(at 138.938 154.178 90)
 			(effects
@@
 	(symbol
 		(lib_id "power:GND")
-		(at 238.76 68.58 0)
+		(at 201.93 -15.24 0)
 		(unit 1)
 		(exclude_from_sim no)
@@
 		(fields_autoplaced yes)
 		(property "Reference" "#PWR011"
-			(at 238.76 74.93 0)
+			(at 201.93 -8.89 0)
 			(effects
 				(font
@@
 		)
 		(property "Value" "GND"
-			(at 238.76 73.66 0)
+			(at 201.93 -10.16 0)
 			(effects
 				(font
@@
 		)
 		(property "Footprint" ""
-			(at 238.76 68.58 0)
+			(at 201.93 -15.24 0)
 			(effects
 				(font
@@
 		)
 		(property "Datasheet" ""
-			(at 238.76 68.58 0)
+			(at 201.93 -15.24 0)
 			(effects
 				(font
@@
 		)
 		(property "Description" "Power symbol creates a global label with name \"GND\" , ground"
-			(at 238.76 68.58 0)
+			(at 201.93 -15.24 0)
 			(effects
 				(font
@@
 		(on_board yes)
 		(dnp no)
-		(property "Reference" "J5"
+		(property "Reference" "J6"
 			(at 119.38 168.9099 0)
 			(effects
@@
 			(project "TRS80M2 50-34 Floppy Adapter"
 				(path "/f29434cd-fd41-45dc-9c32-41e112fe785e"
-					(reference "J5")
+					(reference "J6")
 					(unit 1)
 				)
@@
 			)
 		)
-		(property "Footprint" "GenericComponents:Resistor-.4in"
+		(property "Footprint" "Resistor_THT:R_Axial_DIN0204_L3.6mm_D1.6mm_P7.62mm_Horizontal"
 			(at 138.938 171.958 90)
 			(effects
@@
 		(on_board yes)
 		(dnp no)
-		(property "Reference" "J4"
+		(property "Reference" "J5"
 			(at 119.38 151.1299 0)
 			(effects
@@
 			(project "TRS80M2 50-34 Floppy Adapter"
 				(path "/f29434cd-fd41-45dc-9c32-41e112fe785e"
-					(reference "J4")
+					(reference "J5")
 					(unit 1)
 				)
@@
 			)
 		)
-		(property "Footprint" "GenericComponents:Resistor-.4in"
+		(property "Footprint" "Resistor_THT:R_Axial_DIN0204_L3.6mm_D1.6mm_P7.62mm_Horizontal"
 			(at 138.938 166.878 90)
 			(effects
